Commit message: change

File: carlike/urdf/car_like_description.urdf (robot description, URDF)
Before this commit: robot full_carlike, 13 links, 12 joints
Links:
- link arm_link1: geometry collision box size=0.05 0.05 0.05; visual mesh filename=package://carlike/meshes/arm_link1.STL
- link arm_link2: geometry collision box size=0.05 0.05 0.05; visual mesh filename=package://carlike/meshes/arm_link2.STL
- link base_link: geometry collision box size=0.05 0.05 0.05; visual mesh filename=package://carlike/meshes/base_link.STL
- link camera_link: geometry collision box size=0.05 0.05 0.05; visual mesh filename=package://carlike/meshes/camera_link.STL
- link end_effector_link: geometry collision box size=0.05 0.05 0.05; visual mesh filename=package://carlike/meshes/end_effector_link.STL
- link lidar_link: geometry collision box size=0.05 0.05 0.05; visual mesh filename=package://carlike/meshes/lidar_link.STL

Commit message: change

File: carlike/urdf/car_like_description.urdf (robot description, URDF)
Before this commit: robot full_carlike, 13 links, 12 joints
Links:
- link arm_link1: geometry collision mesh filename=package://carlike/meshes/arm_link1.STL; visual mesh filename=package://carlike/meshes/arm_link1.STL
- link arm_link2: geometry collision mesh filename=package://carlike/meshes/arm_link2.STL; visual mesh filename=package://carlike/meshes/arm_link2.STL
- link base_link: geometry collision mesh filename=package://carlike/meshes/base_link.STL; visual mesh filename=package://carlike/meshes/base_link.STL
- link camera_link: geometry collision mesh filename=package://carlike/meshes/camera_link.STL; visual mesh filename=package://carlike/meshes/camera_link.STL
- link end_effector_link: geometry collision mesh filename=package://carlike/meshes/end_effector_link.STL; visual mesh filename=package://carlike/meshes/end_effector_link.STL
- link lidar_link: geometry collision mesh filename=package://carlike/meshes/lidar_link.STL; visual mesh filename=package://carlike/meshes/lidar_link.STL
